Commit message: update my_robot.xacro
update the camera_optical_joint

File: my_robot/urdf/my_robot.p4.xacro (robot description, xacro)
@@ -8,11 +8,4 @@
     <child link="chassis" />
   </joint>
-  <joint name="camera_optical_joint" type="fixed">
-    <origin xyz="0 0 0" rpy="-1.5707 0 -1.5707"/>
-    <parent link="camera"/>
-    <child link="camera_link_optical"/>
-  </joint>
-  <link name="camera_link_optical">
-  </link>
   <joint name="camera_joint" type="fixed">
     <origin xyz="0.2 0 0" rpy="0 0 0" />
